File: FPGA_FOC_boards/motherboard.sch (EAGLE design)
At the start: 148 parts, among them J1 PRIUS_INV_DB26, U1 ADS7883, U10 ADS7883, U11 ADS7883, U12 ADS7883, U13 LM7321, U14 LM7321, U15 LM7321, U16 LM7321, U17 CD40109BPWR, U18 CD40109BPWR, U19 LM7321, U2 ADS7883, U20 CMOD_A7, U3 ADS7883, U4 ADS7883, U5 LM7321, U6 LM7321, U7 LM7321, U8 LM7321, U9 ADS7883

Commit message: started adding in the resolver hardware onto the motherboard, began ripping up some parts of the v1 board to make room for resolver hardware
Parts:
- added C56, C57: 20p, FPGA_FOC_lib:CAP_SMD_0402
- added C58, C59, C60, C61: 10u, FPGA_FOC_lib:CAP_SMD_0603
- added C62, C63, C64: 10n, FPGA_FOC_lib:CAP_SMD_0402
- added C66, C67, C68, C69: (no value), FPGA_FOC_lib:CAP_SMD_0402
- added H5: BOLTHOLE_M3, FPGA_FOC_lib:BOLTHOLE_M3
- added Q1, Q2, Q5, Q6: (no value), FPGA_FOC_lib:BJT_NPN
- added Q3, Q4, Q7, Q8: (no value), FPGA_FOC_lib:BJT_PNP
- added R53, R54, R55, R56, R57, R58, R61, R62, R63, R64, R65, R66: (no value), FPGA_FOC_lib:RES_SMD_0402
- added R59, R60, R71, R72: 1k, FPGA_FOC_lib:RES_SMD_0402
- added R67, R68, R69, R70: 16, FPGA_FOC_lib:RES_SMD_0805
- added U23: ADS1205, FPGA_FOC_lib:ADS1205
- added U24, U25: LM7321, FPGA_FOC_lib:LM7321
- added Y1: 8.192mHz, FPGA_FOC_lib:LFXTAL061486
- J2: value (none) -> DB09_RA; device FPGA_FOC_lib:M20 -> FPGA_FOC_lib:DB09_RA
- R36: value (none) -> 10k
Connections:
- new net !RD_EXC: R61.1, U23.!EXC
- new net !RD_EXCOUT: C69.2, J2.9, R62.1, R69.2, R70.1
- new net MT1: J2.6
- new net MT2: J2.7
- new net M_CASE: J2.8
- new net Q1_BASE: Q1.B, R55.2, R56.1
- new net Q1_EMITTER: Q1.E, R67.1
- new net Q2_BC: Q2.B, Q2.C, R56.2
- new net Q3_BASE: Q3.B, R57.2, R58.1
- new net Q3_EMITTER: Q3.E, R68.2
- new net Q4_BC: Q4.B, Q4.C, R57.1
- new net Q5_BASE: Q5.B, R63.1, R64.2
- new net Q5_EMITTER: Q5.E, R69.1
- new net Q6_BC: Q6.B, Q6.C, R64.1
- new net Q7_BASE: Q7.B, R65.1, R66.2
- new net Q7_EMITTER: Q7.E, R70.2
- new net Q8_BC: Q8.B, Q8.C, R65.2
- new net RD_CLKIN: C57.1, U23.CLKIN, Y1.X2
- new net RD_COS: J2.1, U23.COS
- new net RD_COSLO: J2.2, U23.COSLO
- new net RD_CPO: U23.CPO
- new net RD_EXC: R53.1, U23.EXC
- new net RD_EXCOUT: C68.2, J2.5, R54.1, R67.2, R68.1
- new net RD_REFBYP: C58.1, U23.REFBYP
- new net RD_SIN: J2.4, U23.SIN
- new net RD_SINLO: J2.3, U23.SINLO
- new net RD_XTALOUT: C56.2, U23.XTALOUT, Y1.X1
- new net U24_IN+: R59.2, R60.1, U24.IN+
- new net U24_IN-: C68.1, R53.2, R54.2, U24.IN-
- new net U24_OUT: Q2.E, Q4.E, U24.OUT
- new net U25_IN+: R71.2, R72.1, U25.IN+
- new net U25_IN-: C69.1, R61.2, R62.2, U25.IN-
- new net U25_OUT: Q6.E, Q8.E, U25.OUT
- net !RD_CS: now also U23.!CS; no longer J2.16
- net !RD_DOS: now also U23.!DOS; no longer J2.4
- net !RD_LOT: now also U23.!LOT; no longer J2.3
- net !RD_RD: now also U23.!RD; no longer J2.17
- net !RD_RDVEL: now also U23.!RDVEL; no longer J2.14
- net !RD_RESET: now also U23.!RESET; no longer J2.2
- net !RD_SAMPLE: now also U23.!SAMPLE; no longer J2.15
- net 12V: now also C66.1, C67.1, Q1.C, Q5.C, R55.1, R63.2, U24.V+, U25.V+; no longer J2.19
- net 5V: now also C59.1, C60.1, C61.1, C62.1, C63.1, C64.1, R59.1, R71.1, U23.AV_DD, U23.DV_DD, U23.FS1, U23.FS2; no longer J2.20
- net GND: now also C56.1, C57.2, C58.2, C59.2, C60.2, C61.2, C62.2, C63.2, C64.2, C66.2, C67.2, H5.P, J2.10, Q3.C, Q7.C, R58.2, R60.2, R66.1, R72.2, U23.!SOE, U23.A_GND, U23.D_GND, U24.V-, U25.V-, Y1.CASE; no longer J2.1, J2.18, J2.9
- net RD_A: now also U23.A; no longer J2.8
- net RD_B: now also U23.B; no longer J2.7
- net RD_DIR: now also U23.DIR; no longer J2.5
- net RD_MT1: no longer J2.11
- net RD_MT2: no longer J2.10
- net RD_NM: now also U23.NM; no longer J2.6
- net RD_SCLK: now also U23.SCLK/DB10; no longer J2.12
- net RD_SO: now also U23.SO/DB11; no longer J2.13
Other:
- note added: "Thoughts from Revision 1: Move away from the 12v reg im currently using, didn't work and was a bother to solder. If for some reason I decide to keep using the 12v reg, make all pads have large vias to the bottom side, to be able to observe if soldered. 12v/15v jumper option maybe, resolver doesn't seem like it needs only 12v, so maybe move to 15v. The 5v reg seemed fine, but was also nontrivial t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"

Commit message: started the CCU board
Parts:
- added C65, C70, C71: 1u, FPGA_FOC_lib:CAP_SMD_0402
- added C72: 10n, FPGA_FOC_lib:CAP_SMD_0402
- added J3, J4: (no value), FPGA_FOC_lib:SM04B-SRSS-TB
- added R32: 120, FPGA_FOC_lib:RES_SMD_0402
- added SJ1: (no value), FPGA_FOC_lib:SOLDERABLE_JUMPER_1POS_NP
- added TP11: !EXCOUT, FPGA_FOC_lib:TESTPOINT_MINI
- added TP12: EXCOUT, FPGA_FOC_lib:TESTPOINT_MINI
- added U26: SN65HVD23X, FPGA_FOC_lib:SN65HVD23X
- C66, C67: value (none) -> 1u
- C68, C69: value (none) -> DNP
- R53, R61: value (none) -> 1k
- R54, R62: value (none) -> 2.4k
- R55, R58, R63, R66: value (none) -> 2.2k
- R56, R57, R64, R65: value (none) -> 3.3
- R59, R71: value 1k -> 10k
- R60, R72: value 1k -> 4.16k
- R67: value 16 -> 4.7k
- R68, R69, R70: value 16 -> 4.7
Connections:
- new net CANH: J3.2, J4.2, R32.1, U26.CANH
- new net CANL: J3.1, J4.1, SJ1.2, U26.CANL
- new net CAN_RS: U26.RS
- new net CAN_RXD: U26.RXD
- new net CAN_TXD: U26.TXD
- new net CAN_VREF: U26.VREF
- new net N$2: R32.2, SJ1.1
- net !RD_EXCOUT: now also TP11.TP
- net 12V: now also C65.1, C70.1, R59.1, R71.1
- net 3.3V: now also C71.1, C72.1, U26.VCC
- net 5V: now also J3.4, J4.4; no longer R59.1, R71.1
- net GND: now also C65.2, C70.2, C71.2, C72.2, J3.3, J4.3, U26.GND
- net RD_EXCOUT: now also TP12.TP
Other:
- note added: "May want to reduce this gain if having rail to rail issues"
- note added: "Populate the parallel capacitors if noise is a problem"
